File: Communication.kicad_sch (KiCad schematic)
At the start: 39 parts, among them IC3 ILD206T, J11 BME280, J13 I/O, J14 Top signals, J15 Fuel cell signals, J4 61200621621, P1 USB_C_Plug_USB2.0, U5 USBLC6-2P6, U7 SN65HVD232

Commit message: Full
Changed lines of the file:
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@@
+	)
+	(junction
+		(at 71.882 155.194)
+		(diameter 0)
+		(color 0 0 0 0)
 	)
 	(junction
@@
 	)
 	(junction
-		(at 71.882 155.194)
-		(diameter 0)
-		(color 0 0 0 0)
-	)
-	(junction
 		(at 65.786 30.988)
 		(diameter 0)
@@
 	(wire
 		(pts
-			(xy 71.882 155.194) (xy 66.802 155.194)
+			(xy 66.802 155.194) (xy 71.882 155.194)
 		)
 		(stroke
@@
 	(wire
 		(pts
-			(xy 80.772 155.194) (xy 71.882 155.194)
+			(xy 75.946 155.194) (xy 71.882 155.194)
 		)
 		(stroke
@@
 		)
 	)
-	(label "Antena"
-		(at 80.772 155.194 180)
-		(effects
-			(font
-				(size 1.27 1.27)
-			)
-			(justify right bottom)
-		)
-	)
 	(label "VBUS"
 		(at 202.692 101.854 180)
@@
 		(effects
 			(font
+				(size 1.27 1.27)
+			)
+			(justify left)
+		)
+	)
+	(hierarchical_label "Antena"
+		(shape input)
+		(at 75.946 155.194 0)
+		(effects
+			(font
