File: FCCU-v21-schematic-pcb.kicad_pcb (KiCad board)
At the start: 4 copper layers, 100 x 100 mm, 280 parts, among them IC1 LM76202QPWPRQ1, IC2 AD8544ARUZ-REEL, IC3 ILD206T, IC4 ADS1015IDGSR, IC5 ADS1015IDGSR, IC6 ADS1015IDGSR, J1 Supercapacitors, J10 M12A-05PMMR-SF7003, J11 BME, J13 I/O, J14 Top signals, J15 Fuel cell signals, J2 CAN, J4 61200621621, J4 P_Valve, J5 FC_ON, J6 FC Module, J69 ADC, Freq, 4-20mA, J7 FC Cooling, J8 M_Valve, P1 USB_C_Plug_USB2.0, Q1 PMPB10XNX, Q2 PMPB10XNX, Q3 PMPB10XNX, Q4 PMPB10XNX, Q5 PMPB10XNX, U1 LM5013DDAR, U2 TPS62933, U3 LDI1117-05H, U4 LDI1117-3.3H, U5 USBLC6-2P6, U6 ESP32-S3FN8, U7 SN65HVD232, Y1 Crystal_40MHz, Y2 9HT7-32.768KDZF-T

Commit message: Full
Parts:
- E_1, E_2, K_1, K_2: moved to F.Cu
- turned E_1 to 180 degrees
- turned E_2 to 180 degrees
- turned K_1 to 180 degrees
- turned K_2 to 0 degrees
Connections:
- D13 pad 2: /IO/PURGE_VALVE -> /IO2/I/O_4
- D14 pad 2: /IO/PURGE_VALVE -> /IO2/I/O_3
- IC2 pad 3: Net-(IC2-+IN_A) -> /IO/TEMP_SENSOR_2
- J6 pad 4: /FC_1V -> /IO/LP_2
- J7 pad 5: /TEMP_SENSOR -> /IO/TEMP_SENSOR_1
- J7 pad 6: /IO/LP_2 -> /IO/TEMP_SENSOR_2
Routing:
- net (no net): track 36.2 -> 24.2 mm
- net /IO/PURGE_VALVE: track 62.9 -> 53.3 mm
- net /IO/LP_2: track 0.00 -> 9.47 mm
- net /IO2/I/O_3: track 31.2 -> 38.2 mm
- net /IO2/I/O_4: track 34.9 -> 39.9 mm
Other:
- board text added: "G T_1"
- board text added: "T_2 +12V"
- board text removed: "G T_R"
- board text removed: "LP_2 +12V"
