File: io2.kicad_sch (KiCad schematic)
At the start: 78 parts, among them IC2 AD8544ARUZ-REEL, IC4 ADS1015IDGSR, IC5 ADS1015IDGSR, IC6 ADS1015IDGSR

Commit message: Full
Changed lines of the file:
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@@
 		)
 	)
-	(hierarchical_label "SCL_MCU"
+	(hierarchical_label "+3.3V"
+		(shape output)
+		(at 14.732 208.026 0)
+		(effects
+			(font
+				(size 1.27 1.27)
+			)
+			(justify left)
+		)
+	)
+	(hierarchical_label "SCL_G34"
 		(shape input)
 		(at 102.362 106.68 0)
@@
 		)
 	)
-	(hierarchical_label "SCL_MCU"
+	(hierarchical_label "SCL_G34"
 		(shape input)
 		(at 222.758 30.48 180)
@@
 		)
 	)
-	(hierarchical_label "SDA_MCU"
+	(hierarchical_label "SDA_G35"
 		(shape input)
 		(at 102.362 109.22 0)
@@
 		)
 	)
-	(hierarchical_label "SCL_MCU"
+	(hierarchical_label "SCL_G34"
 		(shape input)
 		(at 95.25 31.496 180)
@@
 		)
 	)
-	(hierarchical_label "SDA_MCU"
+	(hierarchical_label "SDA_G35"
 		(shape input)
 		(at 94.742 22.606 180)
@@
 		)
 	)
-	(hierarchical_label "SDA_MCU"
+	(hierarchical_label "SDA_G35"
 		(shape input)
 		(at 227.838 41.402 0)
