File: schematc-io.kicad_sch (KiCad schematic)
At the start: 63 parts, among them Q1 PMPB10XNX, Q2 PMPB10XNX, Q3 PMPB10XNX, Q4 PMPB10XNX, Q5 PMPB10XNX, SW1 TL3305BF100QG, SW2 TL3305BF100QG, SW3 TL3305BF100QG

Commit message: Full
Parts:
- renumbered D14 to D13, D13 to D14
Changed lines of the file:
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@@
 		(dnp no)
 		(fields_autoplaced yes)
-		(property "Reference" "D14"
+		(property "Reference" "D13"
 			(at 85.09 159.7025 90)
 			(show_name no)
@@
 			(project "FCCU_v2_schematic-main"
 				(path "/c9ad7189-d3b2-414a-9743-efd8e57cd755/e4695f4d-6fa6-4597-a598-6a2f28a255eb"
-					(reference "D14")
+					(reference "D13")
 					(unit 1)
 				)
@@
 		(dnp no)
 		(fields_autoplaced yes)
-		(property "Reference" "D13"
+		(property "Reference" "D14"
 			(at 84.074 127.1905 90)
 			(show_name no)
@@
 			(project "FCCU_v2_schematic-main"
 				(path "/c9ad7189-d3b2-414a-9743-efd8e57cd755/e4695f4d-6fa6-4597-a598-6a2f28a255eb"
-					(reference "D13")
+					(reference "D14")
 					(unit 1)
 				)
