File: schematic-mcu.kicad_sch (KiCad schematic)
At the start: 32 parts, among them U6 ESP32-S3FN8, Y1 Crystal_40MHz, Y2 9HT7-32.768KDZF-T

Commit message: Full
Changed lines of the file:
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@@
-		)
-	)
-	(label "Antena"
-		(at 111.252 52.578 0)
-		(effects
-			(font
-				(size 1.27 1.27)
-			)
-			(justify left bottom)
 		)
 	)
@@
 		(effects
 			(font
+				(size 1.27 1.27)
+			)
+			(justify right)
+		)
+	)
+	(hierarchical_label "Antena"
+		(shape output)
+		(at 111.252 52.578 180)
+		(effects
+			(font
